File: ccd.sch (KiCad schematic (older format))
At the start: 29 parts, among them P1 CONN_12X2, Q1 NPN, Q4 NPN, Q5 NPN, U1 UPD3798, U2 74HC04, U3 4052

Commit message: Schematics complete
Parts:
- added R? (x2): 10k, symbol R
- added R?: 1k, symbol R
- added R? (x2): 220, symbol R
- renumbered Q1 to Q3
Connections:
- net DGND: now also Q3.1 (E), Q4.1 (E), U3.1 (Y0), U3.2 (Y2), U3.4 (Y3), U3.5 (Y1), U3.6 (Inh), U3.7 (VEE)
- net VDD: now also R?.1, R?.2
- net ADDR_A: now reaches U3.10 (A)
- net ADDR_A: now also Q3.3 (C), R?.2
- net ADDR_B: now reaches U3.9 (B)
- net ADDR_B: now also Q4.3 (C), R?.1
- net Phi_TG1_L: now reaches U2.8
- net Phi_TG1_L: now also R?.1
- net Phi_TG_1_in: now reaches U2.9
- net Phi_TG_1_in: now also P1.16 (P16)
- net Phi_TG23_L: now reaches U2.10
- net Phi_TG23_L: now also R?.1
- net Phi_TG_23_in: now reaches U2.11
- net Phi_TG_23_in: now also P1.18 (P18)
- net at Q3.2 (B): now also R?.2
- net Phi_TG23: now reaches U1.10 (Phi_TG3)
- net Phi_TG23: now also U1.22 (Phi_TG2), R?.2
- net Phi_TG1: now reaches U1.23 (Phi_TG1)
- net Phi_TG1: now also R?.2
- net ADDR_A_inv: now reaches P1.6 (P6)
- net ADDR_A_inv: now also R?.1
- net FOO_5 renamed ADDR_B_inv
- no-connect marks 17 -> 18
Other:
- moved on the sheet: Q3, Q4, R?

Commit message: Final schematics. Added the kicad .pro file. Started writing the arduino source code. Still missing: Analog-Digital conversion (including sending the results via uart), pin definitions.
Connections:
- net FOO_21 renamed V_out
- no-connect marks 18 -> 30
Other:
- note added: "(probably)"
- note added: "(probably)\n"
Changed lines of the file:
@@
-EESchema Schematic File Version 2  date Sat 14 Apr 2012 09:21:16 PM CEST
+EESchema Schematic File Version 2  date Sat 14 Apr 2012 09:36:54 PM CEST
 LIBS:power
 LIBS:device
@@
 Comment4 ""
 $EndDescr
+Text Notes 2050 5250 1    60   ~ 0
+(probably)
+Text Notes 2250 5250 1    60   ~ 0
+(probably)
+NoConn ~ 2250 5300
+Text Notes 5500 3100 0    60   ~ 0
+(probably)\n
+NoConn ~ 5650 2950
+NoConn ~ 2450 4800
+NoConn ~ 2850 4800
+NoConn ~ 2750 4800
+NoConn ~ 2250 6700
+NoConn ~ 2450 6700
+NoConn ~ 2750 6700
+NoConn ~ 2850 6700
+NoConn ~ 1950 6700
+NoConn ~ 1850 6700
+NoConn ~ 1750 6700
 Wire Wire Line
 	5750 3750 5750 3650
@@
 	1900 2400 1900 2100
 Wire Wire Line
-	2150 6100 2150 6600
+	2150 6100 2150 6700
 Wire Wire Line
 	4350 6000 3850 6000
 Wire Wire Line
-	2650 6100 2650 6600
+	2650 6100 2650 6700
 Wire Wire Line
 	5350 1500 5250 1500
@@
 	4350 4650 3950 4650
 Wire Wire Line
-	2350 6100 2350 6600
+	2350 6100 2350 6700
 Wire Wire Line
 	5250 4650 5650 4650
@@
 	2600 4000 2600 4300
 Wire Wire Line
-	1850 5300 1850 5000
+	1850 5300 1850 4800
 Connection ~ 7350 2250
 Wire Wire Line
@@
 	2200 4000 2200 4300
 Wire Wire Line
-	1750 6100 1750 6400
-Wire Wire Line
-	1750 5300 1750 5000
-Wire Wire Line
-	2450 6100 2450 6400
-Wire Wire Line
-	2750 5300 2750 5000
-Wire Wire Line
-	2550 5300 2550 5000
-Wire Wire Line
-	2250 6100 2250 6400
-Wire Wire Line
-	1850 6100 1850 6400
-Wire Wire Line
-	1950 6100 1950 6400
+	1750 6100 1750 6700
+Wire Wire Line
+	1750 5300 1750 4800
+Wire Wire Line
+	2450 6100 2450 6700
+Wire Wire Line
+	2750 5300 2750 4800
+Wire Wire Line
+	2550 5300 2550 4800
+Wire Wire Line
+	2250 6100 2250 6700
+Wire Wire Line
+	1850 6100 1850 6700
+Wire Wire Line
+	1950 6100 1950 6700
 Wire Wire Line
 	2100 4000 2100 4300
@@
 	6150 4650 6450 4650
 Wire Wire Line
-	1950 5300 1950 5000
+	1950 5300 1950 4800
 Wire Wire Line
 	1500 7400 1500 7300
@@
 	4350 6450 3950 6450
 Wire Wire Line
-	2550 6100 2550 6600
+	2550 6100 2550 6700
 Wire Wire Line
 	2850 5300 2850 4800
@@
 	10400 5400 10000 5400
 Wire Wire Line
-	2750 6100 2750 6600
+	2750 6100 2750 6700
 Wire Wire Line
 	6950 5400 6850 5400
@@
 	4750 1500 4250 1500
 Wire Wire Line
-	2050 6100 2050 6600
+	2050 6100 2050 6700
 Wire Wire Line
 	4350 5550 3850 5550
@@
 Text Label 2000 2100 3    60   ~ 0
 Phi_TG1
-Text Label 2150 6600 1    60   ~ 0
+Text Label 2150 6700 1    60   ~ 0
 Phi_TG_1_in
 Text Label 3850 5550 0    60   ~ 0
@@
 Text Label 3850 6000 0    60   ~ 0
 Phi_TG_23_in
-Text Label 2050 6600 1    60   ~ 0
+Text Label 2050 6700 1    60   ~ 0
 Phi_TG_23_in
 NoConn ~ 2050 5300
-Text Label 2650 6600 1    60   ~ 0
+Text Label 2650 6700 1    60   ~ 0
 ADDR_A_inv
 Text Label 4250 1500 0    60   ~ 0
@@
 	0    -1   -1   0
 $EndComp
-Text Label 2750 6600 1    60   ~ 0
+Text Label 2750 6700 1    60   ~ 0
 photo_out
 Text Label 9500 5400 2    60   ~ 0
@@
 Text Label 2350 4800 3    60   ~ 0
 Phi_1_in
-Text Label 2550 6600 1    60   ~ 0
+Text Label 2550 6700 1    60   ~ 0
 Phi_2_in
 $Comp
@@
 	0    -1   -1   0
 $EndComp
-Text Label 2350 6600 1    60   ~ 0
+Text Label 2350 6700 1    60   ~ 0
 Phi_RB_in
 Text Label 3950 4200 0    60   ~ 0
@@
 Text Label 1200 6900 0    60   ~ 0
 VDD_in
-Text Label 1950 5000 3    60   ~ 0
+Text Label 1950 4800 3    60   ~ 0
 VDD_in
 Text Label 6450 4200 2    60   ~ 0
@@
 Text Label 2600 4300 1    60   ~ 0
 Phi_CLB
-Text Label 1850 5000 3    60   ~ 0
-FOO_21
+Text Label 1850 4800 3    60   ~ 0
+V_out
 Text Label 7050 2800 2    60   ~ 0
-FOO_21
+V_out
 $Comp
 L VDD #PWR10
@@
 Text Label 2200 2100 3    60   ~ 0
 Phi_2
-Text Label 1750 5000 3    60   ~ 0
+Text Label 1750 4800 3    60   ~ 0
 AGND
-Text Label 1750 6400 1    60   ~ 0
+Text Label 1750 6700 1    60   ~ 0
 AGND
-Text Label 1850 6400 1    60   ~ 0
+Text Label 1850 6700 1    60   ~ 0
 AGND
-Text Label 1950 6400 1    60   ~ 0
+Text Label 1950 6700 1    60   ~ 0
 AGND
-Text Label 2750 5000 3    60   ~ 0
+Text Label 2750 4800 3    60   ~ 0
 DGND
-Text Label 2550 5000 3    60   ~ 0
+Text Label 2550 4800 3    60   ~ 0
 DGND
-Text Label 2450 6400 1    60   ~ 0
+Text Label 2450 6700 1    60   ~ 0
 DGND
-Text Label 2250 6400 1    60   ~ 0
+Text Label 2250 6700 1    60   ~ 0
 DGND
 $Comp

Commit message: Fixed a bug in the schematics: The device actually takes both 5V and 12V supplies. The inputs operate on a 5V logic level, the analog output goes up to 12.
Connections:
- net VCC_photo is gone; now on net 5V_logic: C?.1, P1.9 (P9), R?.1, R?.2
- net 5V_logic: now reaches P1.13 (P13)
- no-connect marks 30 -> 28
